File: BitRex.kicad_pcb (KiCad board)
At the start: 6 copper layers, 95 x 190 mm, 327 parts, among them J1 Connector 02x01, J4 Conn_01x06, M1 Fan_4pin, M2 Fan_4pin, U1 TPS53647, U10 BM1373, U11 BM1373, U12 BM1373, U13 BM1373, U14 TXU0304PW, U15 T-Display-S3, U16 EMC2302-1, U17 TXU0102-DCU, U18 TMP1075, U19 TMP1075, U2 AP3211, U20 TLV75733PDBVR, U3 MCP1824T-0802E, U4 MCP1824T-1202E, U5 CSD95472Q5MC, U6 CSD95472Q5MC, U7 CSD95472Q5MC, U8 CSD95472Q5MC, U9 25MHz

Commit message: Add files via upload
Parts:
- removed D3: 1N5819-No need, Diode_SMD:D_SOD-123
- removed JP3: SolderJumper_2_Open, Jumper:SolderJumper-2_P1.3mm_Open_RoundedPad1.0x1.5mm
- R1: value 100k -> 66.5k
Routing:
- net +VRef: track 246.9 -> 253.0 mm
- net unconnected-(U15-5V-Pad12): track 4.40 -> 0.00 mm
- net +5V: track 314.8 -> 310.8 mm
- net +3V3: track 323.1 -> 325.9 mm, vias 13 -> 15
- net Net-(D3-A): track 1.99 -> 0.00 mm
- net /BM1373/TXD: track 32.1 -> 32.9 mm
- net /BM1373/RXD: track 33.7 -> 34.4 mm
- net +12V: track 101.1 -> 100.5 mm
- net GND: vias 513 -> 515
