File: pi.kicad_sch (KiCad schematic)
At the start: 19 parts, among them M1 Fan_4pin, M2 Fan_4pin, U15 T-Display-S3, U16 EMC2302-1, U17 TXU0102-DCU, U18 TMP1075, U19 TMP1075

Commit message: Add files via upload
Parts:
- removed D3: 1N5819-No need, Diode_SMD:D_SOD-123, symbol Diode:US1D
- removed JP3: SolderJumper_2_Open, Jumper:SolderJumper-2_P1.3mm_Open_RoundedPad1.0x1.5mm, symbol Jumper:SolderJumper_2_Open
Connections:
- no-connect marks 9 -> 10
