File: power.kicad_sch (KiCad schematic)
At the start: 196 parts, among them J2 Conn_01x01, J3 Conn_01x01, U1 TPS53647, U2 AP3211, U20 TLV75733PDBVR, U3 MCP1824T-0802E, U4 MCP1824T-1202E, U5 CSD95472Q5MC, U6 CSD95472Q5MC, U7 CSD95472Q5MC, U8 CSD95472Q5MC

Commit message: Add files via upload
Parts:
- R1: value 100k -> 66.5k
Changed lines of the file:
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@@
 			)
 		)
-		(property "Value" "100k"
+		(property "Value" "66.5k"
 			(at 37.592 91.44 90)
 			(show_name no)
